File: 690 module pico.kicad_sch (KiCad schematic)
At the start: 12 parts, among them J1 Conn_01x04_Male, J2 USB_B_Micro, SW1 Bootsel, SW2 Reset, U1 USBLC6-2P6, U2 DA14695_000HQ2

Commit message: Ordered version 1
Parts:
- added TP1: Vbat, TestPoint:TestPoint_Pad_1.0x1.0mm_custom, symbol Connector:TestPoint_Alt
- added TP2: Vbus, TestPoint:TestPoint_Pad_1.0x1.0mm_custom, symbol Connector:TestPoint_Alt
- added TP3: USB_P, TestPoint:TestPoint_Pad_1.0x1.0mm_custom, symbol Connector:TestPoint_Alt
- added TP4: USB_N, TestPoint:TestPoint_Pad_1.0x1.0mm_custom, symbol Connector:TestPoint_Alt
- added TP5: UART_TX, TestPoint:TestPoint_Pad_1.0x1.0mm_custom, symbol Connector:TestPoint_Alt
- added TP6: UART_RX, TestPoint:TestPoint_Pad_1.0x1.0mm_custom, symbol Connector:TestPoint_Alt
- added TP7: ~{Bootsel}, TestPoint:TestPoint_Pad_1.0x1.0mm_custom, symbol Connector:TestPoint_Alt
- added TP8: ~{RST}, TestPoint:TestPoint_Pad_1.0x1.0mm_custom, symbol Connector:TestPoint_Alt
- added TP9: GND, TestPoint:TestPoint_Pad_1.0x1.0mm_custom, symbol Connector:TestPoint_Alt
Connections:
- net +BATT: now also TP1.1
- net GND: now also TP9.1
- net UART_RX: now also TP6.1
- net UART_TX: now also TP5.1
- net USB_N: now also TP4.1
- net USB_P: now also TP3.1
- net VBUS: now also TP2.1
- net RST renamed ~{RST}
- net ~{RST}: now also TP8.1
- net bootsel renamed ~{Bootsel}
- net ~{Bootsel}: now also TP7.1
Other:
- moved on the sheet: B1, J1, U2A, U2B

Commit message: Add order files and replace USB connector
Parts:
- J2: LCSC partnumber C381144 -> C404969
Changed lines of the file:
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@@
       (effects (font (size 1.27 1.27)) hide)
     )
-    (property "LCSC partnumber" "C381144" (id 4) (at 35.56 63.5 0)
+    (property "LCSC partnumber" "C404969" (id 4) (at 35.56 63.5 0)
       (effects (font (size 1.27 1.27)) hide)
     )
